Commit message: Urdf fake imus

File: go1_description/urdf/go1_slip_stack.urdf (robot description, URDF)
Before this commit: robot go1, 46 links, 45 joints
Joints:
- joint FL_foot_fixed: axis (none) -> 1 0 0; limit (none) -> lower=-0.863 upper=0.863 effort=23.7 velocity=30.1; type fixed -> revolute
- joint FR_foot_fixed: axis (none) -> 1 0 0; limit (none) -> lower=-0.863 upper=0.863 effort=23.7 velocity=30.1; type fixed -> revolute
- joint RL_foot_fixed: axis (none) -> 1 0 0; limit (none) -> lower=-0.863 upper=0.863 effort=23.7 velocity=30.1; type fixed -> revolute
- joint RR_foot_fixed: axis (none) -> 1 0 0; limit (none) -> lower=-0.863 upper=0.863 effort=23.7 velocity=30.1; type fixed -> revolute
